Commit message: justina_simple.urdf con color, colision e inercia. Programa para mover joint en gazebo

File: catkin_ws/src/hardware/robot_description/models/justina_simple.urdf (robot description, URDF)
Before this commit: robot justina_simple, 34 links, 33 joints
Links:
- link head_link1: geometry collision box size=0.04 0.04 0.2; visual box size=0.04 0.04 0.2
- link head_link2: geometry collision box size=0.03 0.03 0.03; visual box size=0.03 0.03 0.03
- link kinect_link: geometry collision box size=0.058 0.207 0.04; visual box size=0.058 0.207 0.04
- link left_arm_grip_center: geometry collision box size=0.04 0.1 0.04; visual box size=0.04 0.1 0.04
- link left_arm_grip_left: geometry collision box size=0.13 0.015 0.03; visual box size=0.13 0.015 0.03
- link left_arm_grip_right: geometry collision box size=0.13 0.015 0.03; visual box size=0.13 0.015 0.03
- link left_arm_link1: geometry collision box size=0.07 0.08 0.05; visual box size=0.07 0.08 0.05
- link left_arm_link2: geometry collision box size=0.21 0.04 0.04; visual box size=0.21 0.04 0.04
- link left_arm_link3: geometry collision box size=0.075 0.05 0.05; visual box size=0.075 0.05 0.05
- link left_arm_link4: geometry collision box size=0.18 0.04 0.04; visual box size=0.18 0.04 0.04
- link left_arm_link5: geometry collision box size=0.045 0.05 0.05; visual box size=0.045 0.05 0.05
- link left_arm_link6: geometry collision box size=0.1 0.04 0.04; visual box size=0.1 0.04 0.04
- link left_arm_link7: geometry collision box size=0.06 0.04 0.04; visual box size=0.06 0.04 0.04
- link right_arm_grip_center: geometry collision box size=0.04 0.1 0.04; visual box size=0.04 0.1 0.04
- link right_arm_grip_left: geometry collision box size=0.13 0.015 0.03; visual box size=0.13 0.015 0.03
- link right_arm_grip_right: geometry collision box size=0.13 0.015 0.03; visual box size=0.13 0.015 0.03
- link right_arm_link1: geometry collision box size=0.07 0.08 0.05; visual box size=0.07 0.08 0.05
- link right_arm_link2: geometry collision box size=0.21 0.04 0.04; visual box size=0.21 0.04 0.04
- link right_arm_link3: geometry collision box size=0.075 0.05 0.05; visual box size=0.075 0.05 0.05
- link right_arm_link4: geometry collision box size=0.18 0.04 0.04; visual box size=0.18 0.04 0.04
- link right_arm_link5: geometry collision box size=0.045 0.05 0.05; visual box size=0.045 0.05 0.05
- link right_arm_link6: geometry collision box size=0.1 0.04 0.04; visual box size=0.1 0.04 0.04
- link right_arm_link7: geometry collision box size=0.06 0.04 0.04; visual box size=0.06 0.04 0.04
